Commit message: fix: camara en web
se muestra imagen de la camara en la web

File: roberto_mundo/urdf/turtlebot3_burger.urdf (robot description, URDF)
Before this commit: robot turtlebot3_burger, 7 links, 6 joints
Links:
- added link camera_link; collision box size=0.015 0.030 0.027
- added link camera_rgb_frame
- added link camera_rgb_optical_frame
Joints:
- added joint camera_joint: type fixed, parent base_link, child camera_link, origin xyz=0.040 -0.000 0.110 rpy=0 0 0
- added joint camera_rgb_joint: type fixed, parent camera_link, child camera_rgb_frame, origin xyz=0.003 0.000 0.009 rpy=0 0 0
- added joint camera_rgb_optical_joint: type fixed, parent camera_rgb_frame, child camera_rgb_optical_frame, origin xyz=0 0 0 rpy=-1.5707 0 -1.57
